File: logic-power-management-board/logic-power-management-board.kicad_pcb (KiCad board)
At the start: 2 copper layers, 0 parts

Commit message: PCB完成(ビア、シルクを除く)
Parts:
- added C1: 0.1uf, Capacitor_SMD:C_0603_1608Metric_Pad1.08x0.95mm_HandSolder, F.Cu at (35.9, 35.1)
- added C10: 0.1u, Capacitor_SMD:C_0603_1608Metric_Pad1.08x0.95mm_HandSolder, F.Cu at (59.8, 55.4)
- added C11: 0.1u, Capacitor_SMD:C_0603_1608Metric_Pad1.08x0.95mm_HandSolder, F.Cu at (62.0, 81.0)
- added C12: 0.1u, Capacitor_SMD:C_0603_1608Metric_Pad1.08x0.95mm_HandSolder, F.Cu at (54.8, 76.2)
- added C2: 0.1uf, Capacitor_SMD:C_0603_1608Metric_Pad1.08x0.95mm_HandSolder, F.Cu at (35.9, 52.0)
- added C3: 0.1uf, Capacitor_SMD:C_0603_1608Metric_Pad1.08x0.95mm_HandSolder, F.Cu at (35.9, 68.9)
- added C4: 1000μF35V, Capacitor_THT:CP_Radial_D12.5mm_P5.00mm, F.Cu at (57.2, 32.9)
- added C5: 0.1u, Capacitor_SMD:C_0603_1608Metric_Pad1.08x0.95mm_HandSolder, F.Cu at (45.6, 72.0)
- added C6: 0.47u, Capacitor_SMD:C_0603_1608Metric_Pad1.08x0.95mm_HandSolder, F.Cu at (48.2, 68.2)
- added C7: 0.1u, Capacitor_SMD:C_0603_1608Metric_Pad1.08x0.95mm_HandSolder, F.Cu at (52.0, 62.5)
- added C8: 0.1u, Capacitor_SMD:C_0603_1608Metric_Pad1.08x0.95mm_HandSolder, F.Cu at (53.0, 66.0)
- added C9: 0.1u, Capacitor_SMD:C_0603_1608Metric_Pad1.08x0.95mm_HandSolder, F.Cu at (62.8, 56.3)
- added D1: LED, LED_SMD:LED_0603_1608Metric_Pad1.05x0.95mm_HandSolder, F.Cu at (33.4, 81.6)
- added D10: LED, LED_SMD:LED_0603_1608Metric_Pad1.05x0.95mm_HandSolder, F.Cu at (27.0, 83.8)
- added D2: LED, LED_SMD:LED_0603_1608Metric_Pad1.05x0.95mm_HandSolder, F.Cu at (35.0, 81.6)
- added D3: LED, LED_SMD:LED_0603_1608Metric_Pad1.05x0.95mm_HandSolder, F.Cu at (36.6, 81.6)
- added D4: LED, LED_SMD:LED_0603_1608Metric_Pad1.05x0.95mm_HandSolder, F.Cu at (38.2, 81.6)
- added D5: LED, LED_SMD:LED_0603_1608Metric_Pad1.05x0.95mm_HandSolder, F.Cu at (65.6, 81.7)
- added D6: LED, LED_SMD:LED_0603_1608Metric_Pad1.05x0.95mm_HandSolder, F.Cu at (64.0, 81.6)
- added D7: LED, LED_SMD:LED_0603_1608Metric_Pad1.05x0.95mm_HandSolder, F.Cu at (27.0, 79.0)
- added D8: LED, LED_SMD:LED_0603_1608Metric_Pad1.05x0.95mm_HandSolder, F.Cu at (27.0, 80.6)
- added D9: LED, LED_SMD:LED_0603_1608Metric_Pad1.05x0.95mm_HandSolder, F.Cu at (27.0, 82.2)
- added IC1: MCP2562, 0Ikedalibrary:SOIC127P600X175-8N, F.Cu at (57.3, 80.8)
- added J1: Conn_01x02, 0Ikedalibrary:AMASS_XT60PW-M_1x02_P7.20mm_Horizontal, F.Cu at (31.4, 36.7)
- added J2: Conn_01x02, 0Ikedalibrary:AMASS_XT60PW-M_1x02_P7.20mm_Horizontal, F.Cu at (31.4, 53.6)
- added J3: Conn_01x02, 0Ikedalibrary:AMASS_XT60PW-M_1x02_P7.20mm_Horizontal, F.Cu at (31.4, 70.5)
- added J4: Conn_01x02, 0Ikedalibrary:AMASS_XT60PW-F_1x02_P7.20mm_Horizontal, F.Cu at (67.3, 36.7)
- added J5: Conn_01x02, 0Ikedalibrary:AMASS_XT60PW-F_1x02_P7.20mm_Horizontal, F.Cu at (67.3, 70.5)
- added J6: Conn_01x04_Pin, Connector_PinHeader_2.54mm:PinHeader_1x04_P2.54mm_Vertical, F.Cu at (53.8, 70.0)
- added J7: Conn_01x04, Connector_JST:JST_XH_S4B-XH-A_1x04_P2.50mm_Horizontal, B.Cu at (50.9, 75.3)
- added J8: Conn_01x04, Connector_JST:JST_XH_S4B-XH-A_1x04_P2.50mm_Horizontal, B.Cu at (64.5, 75.3)
- added J9: Conn_01x04, Connector_JST:JST_XH_B4B-XH-A_1x04_P2.50mm_Vertical, F.Cu at (61.8, 47.8)
- added Q1: RS6L120BGTB1, 0Ikedalibrary:SOP_Advance, F.Cu at (40.3, 30.5)
- added Q2: RS6L120BGTB1, 0Ikedalibrary:SOP_Advance, F.Cu at (40.3, 47.4)
- added Q3: RS6L120BGTB1, 0Ikedalibrary:SOP_Advance, F.Cu at (40.3, 64.3)
- added R1: 100k, Resistor_SMD:R_0603_1608Metric_Pad0.98x0.95mm_HandSolder, F.Cu at (37.6, 37.8)
- added R10: 120, Resistor_SMD:R_0603_1608Metric_Pad0.98x0.95mm_HandSolder, F.Cu at (48.4, 79.4)
- added R11: 1k, Resistor_SMD:R_0603_1608Metric_Pad0.98x0.95mm_HandSolder, F.Cu at (33.4, 78.2)
- added R12: 1k, Resistor_SMD:R_0603_1608Metric_Pad0.98x0.95mm_HandSolder, F.Cu at (35.0, 78.2)
- added R13: 1k, Resistor_SMD:R_0603_1608Metric_Pad0.98x0.95mm_HandSolder, F.Cu at (36.6, 78.2)
- added R14: 1k, Resistor_SMD:R_0603_1608Metric_Pad0.98x0.95mm_HandSolder, F.Cu at (38.2, 78.2)
- added R15: 1k, Resistor_SMD:R_0603_1608Metric_Pad0.98x0.95mm_HandSolder, F.Cu at (65.6, 78.2)
- added R16: 1k, Resistor_SMD:R_0603_1608Metric_Pad0.98x0.95mm_HandSolder, F.Cu at (64.0, 78.2)
- added R17: 1k, Resistor_SMD:R_0603_1608Metric_Pad0.98x0.95mm_HandSolder, F.Cu at (30.4, 79.0)
- added R18: 1k, Resistor_SMD:R_0603_1608Metric_Pad0.98x0.95mm_HandSolder, F.Cu at (30.4, 80.6)
- added R19: 1k, Resistor_SMD:R_0603_1608Metric_Pad0.98x0.95mm_HandSolder, F.Cu at (30.4, 82.2)
- added R2: 10k, Resistor_SMD:R_0603_1608Metric_Pad0.98x0.95mm_HandSolder, F.Cu at (37.6, 39.4)
- added R20: 1k, Resistor_SMD:R_0603_1608Metric_Pad0.98x0.95mm_HandSolder, F.Cu at (30.4, 83.8)
- added R3: 100k, Resistor_SMD:R_0603_1608Metric_Pad0.98x0.95mm_HandSolder, F.Cu at (37.6, 54.7)
- added R4: 10k, Resistor_SMD:R_0603_1608Metric_Pad0.98x0.95mm_HandSolder, F.Cu at (37.6, 56.3)
- added R5: 100k, Resistor_SMD:R_0603_1608Metric_Pad0.98x0.95mm_HandSolder, F.Cu at (37.6, 71.6)
- added R6: 10k, Resistor_SMD:R_0603_1608Metric_Pad0.98x0.95mm_HandSolder, F.Cu at (37.6, 73.2)
- added R7: 100k, Resistor_SMD:R_0603_1608Metric_Pad0.98x0.95mm_HandSolder, F.Cu at (52.6, 55.6)
- added R8: 10k, Resistor_SMD:R_0603_1608Metric_Pad0.98x0.95mm_HandSolder, F.Cu at (52.6, 57.2)
- added R9: 10k, Resistor_SMD:R_0603_1608Metric_Pad0.98x0.95mm_HandSolder, F.Cu at (64.4, 56.3)
- added REF**: MountingHole_3.2mm_M3, MountingHole:MountingHole_3.2mm_M3, F.Cu at (71.0, 19.0)
- added REF**: MountingHole_3.2mm_M3, MountingHole:MountingHole_3.2mm_M3, F.Cu at (19.0, 19.0)
- added REF**: MountingHole_3.2mm_M3, MountingHole:MountingHole_3.2mm_M3, F.Cu at (19.0, 81.0)
- added REF**: MountingHole_3.2mm_M3, MountingHole:MountingHole_3.2mm_M3, F.Cu at (71.0, 81.0)
- added SW1: SW_Push, 0Ikedalibrary:switch_TVAF06-A020B-R, F.Cu at (55.4, 53.0)
- added SW2: SW_SPDT_312, 0Ikedalibrary:CJS1200A1, F.Cu at (51.4, 80.2)
- added U1: LM5050-1, Package_TO_SOT_SMD:TSOT-23-6, F.Cu at (38.8, 35.1)
- added U2: LM5050-1, Package_TO_SOT_SMD:TSOT-23-6, F.Cu at (38.8, 52.0)
- added U3: LM5050-1, Package_TO_SOT_SMD:TSOT-23-6, F.Cu at (38.8, 68.9)
- added U4: NJM12888F33, Package_TO_SOT_SMD:SOT-23-5_HandSoldering, F.Cu at (48.2, 71.4)
- added U5: STM32G431K8Tx, Package_QFP:LQFP-32_7x7mm_P0.8mm, F.Cu at (58.2, 61.4)
Routing:
- net OUT: track 0.00 -> 98.4 mm
- net +3.3V: track 0.00 -> 82.8 mm, vias 0 -> 1
- net IN1: track 0.00 -> 67.5 mm
- net IN2: track 0.00 -> 52.0 mm, vias 0 -> 2
- net +5V: track 0.00 -> 43.4 mm, vias 0 -> 1
- net IN3: track 0.00 -> 36.2 mm, vias 0 -> 5
- net CANL: track 0.00 -> 32.2 mm, vias 0 -> 1
- net ADC1_CH1: track 0.00 -> 31.8 mm, vias 0 -> 2
- net LED1: track 0.00 -> 30.4 mm, vias 0 -> 2
- net ADC1_CH3: track 0.00 -> 28.7 mm, vias 0 -> 2
- net LED2: track 0.00 -> 28.3 mm, vias 0 -> 2
- net CANH: track 0.00 -> 28.2 mm
- net LED3: track 0.00 -> 26.2 mm, vias 0 -> 2
- net LED4: track 0.00 -> 23.9 mm, vias 0 -> 2
- net ADC1_CH2: track 0.00 -> 22.0 mm, vias 0 -> 2
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- added copper zone on B.Cu, net GNDD
- added copper zone on F.Cu, net GNDD
- added copper zone on B.Cu, net IN1
- added copper zone on F.Cu, net IN1
- added copper zone on B.Cu, net IN2
- added copper zone on F.Cu, net IN2
- added copper zone on B.Cu, net IN3
- added copper zone on F.Cu, net IN3
- added copper zone on F.Cu, net OUT
Other:
- board outline added: 60 x 70 mm
- board text added: "1 2 3 4"
- board text added: "10A"
- board text added: "3.3 5"
- board text added: "5A"
- board text added: "DIO G CLK 3.3"
- board text added: "G T 3.3 R"
- board text added: "H 5 L G"
- board text added: "IN1 IN2 IN3 OUT"
- board text added: "NRST"
- board text added: "入力 → 出力"
