File: switchboard/switchboard.kicad_pcb (KiCad board)
At the start: 2 copper layers, 80 x 40 mm, 16 parts, among them J1 Conn_01x02, J2 Conn_01x02, K1 G8ND-2-DC12SK, SW1 SW_Push_LED, U1 NJM7812SDL1

Commit message: ガーバ生成
Parts:
- added G***: LOGO, LOGO, F.Cu at (79.0, 19.0)
Routing:
- net VCC: vias 0 -> 7
- net OUT: vias 0 -> 5
- net GND: vias 1 -> 54
Other:
- board text added: "create by ikeda"
- board text added: "switchboard version 1.0"
